File: hardware/miñon/aguante/aguante.kicad_pcb (KiCad board)
At the start: 2 copper layers, 20 parts, among them J2 bateria, J3 MPU6050(giro), J5 MT3608(step-up Y CARGA), J6 DFPlayer(audio)

Commit message: Add files via upload
Parts:
- moved C1 101.0 mm to (93.1, 122.8)
- moved R1 95.5 mm to (105.5, 115.0)
- moved R2 94.1 mm to (101.5, 117.5)
- moved R3 82.9 mm to (105.5, 104.5)
- moved R4 82.0 mm to (101.5, 107.0)
- moved C2 74.3 mm to (93.1, 72.1)
- moved C3 74.1 mm to (60.4, 106.3)
- moved J3 74.1 mm to (62.9, 107.3)
- moved J6 74.1 mm to (63.4, 101.9)
- moved R5 74.1 mm to (105.5, 94.0)
- moved C4 73.9 mm to (62.6, 85.3)
- moved U1 73.6 mm to (81.5, 97.1)
- moved J2 73.4 mm to (63.9, 76.5)
- moved J5 73.4 mm to (63.9, 81.3)
- moved JP1 73.4 mm to (58.9, 74.0)
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Routing:
- net +3.3V: track 162.4 -> 134.9 mm
- net +5V: track 84.7 -> 69.6 mm
- net GND: track 50.3 -> 59.7 mm
- net /dedo1: track 19.6 -> 17.5 mm
- net scl: track 7.01 -> 7.92 mm
- net /dedo2: track 16.5 -> 15.7 mm
- net txDFPlayer: track 5.00 -> 5.77 mm
- net rxDFPlayer: track 5.00 -> 5.77 mm
